File: PCB/hackpad - Copy.kicad_pcb (KiCad board)
At the start: 2 copper layers, 85 x 44 mm, 18 parts, among them SW1 SW_Push_45deg, SW2 SW_Push_45deg, SW3 SW_Push_45deg, SW4 SW_Push_45deg, SW5 SW_Push_45deg, SW6 SW_Push_45deg, SW7 RotaryEncoder_Switch, U1 MOUDLE-SEEEDUINO-XIAO

Commit message: yay
Parts:
- SW1, SW2, SW3, SW4, SW5, SW6: footprint Library:SW_Cherry_MX_1.00u_PCB_model -> Button_Switch_Keyboard:SW_Cherry_MX_1.00u_PCB
Other:
- board size 85 x 44 mm -> 185.5 x 44 mm
Changed lines of the file:
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@@
 	(net 19 "unconnected-(U1-PB09_A7_D7_RX-Pad8)")
 	(net 20 "unconnected-(U1-3V3-Pad12)")
-	(footprint "Library:SW_Cherry_MX_1.00u_PCB_model"
+	(footprint "Button_Switch_Keyboard:SW_Cherry_MX_1.00u_PCB"
 		(layer "F.Cu")
 		(at 57.15 38.1)
@@
 			)
 		)
-		(property "Datasheet" ""
+		(property "Datasheet" "~"
 			(at 0 0 0)
 			(unlocked yes)
@@
 			)
 		)
-		(property "Description" ""
+		(property "Description" "Push button switch, normally open, two pins, 45° tilted"
 			(at 0 0 0)
 			(unlocked yes)
@@
 		)
 		(embedded_fonts no)
-		(model "${KICAD9_3DMODEL_DIR}/Button_Switch_THT.3dshapes/Cherry MX.STEP"
+		(model "${KICAD9_3DMODEL_DIR}/Button_Switch_Keyboard.3dshapes/SW_Cherry_MX_1.00u_PCB.step"
 			(offset
-				(xyz -2.5 -4 0)
+				(xyz 0 0 0)
 			)
 			(scale
@@
 			)
 			(rotate
-				(xyz -90 -0 -0)
+				(xyz 0 0 0)
 			)
 		)
 	)
-	(footprint "Library:SW_Cherry_MX_1.00u_PCB_model"
+	(footprint "Button_Switch_Keyboard:SW_Cherry_MX_1.00u_PCB"
 		(layer "F.Cu")
 		(at 57.15 57.15)
@@
 			)
 		)
-		(property "Datasheet" ""
+		(property "Datasheet" "~"
 			(at 0 0 0)
 			(unlocked yes)
@@
 			)
 		)
-		(property "Description" ""
+		(property "Description" "Push button switch, normally open, two pins, 45° tilted"
 			(at 0 0 0)
 			(unlocked yes)
@@
 		)
 		(embedded_fonts no)
-		(model "${KICAD9_3DMODEL_DIR}/Button_Switch_THT.3dshapes/Cherry MX.STEP"
+		(model "${KICAD9_3DMODEL_DIR}/Button_Switch_Keyboard.3dshapes/SW_Cherry_MX_1.00u_PCB.step"
 			(offset
-				(xyz -2.5 -4 0)
+				(xyz 0 0 0)
 			)
 			(scale
@@
 			)
 			(rotate
-				(xyz -90 -0 -0)
+				(xyz 0 0 0)
 			)
 		)
@@
 		)
 		(embedded_fonts no)
-		(model "C:/Kicad_Extra/EC11 Rotary Encoder Dode Switch-15mm .STEP"
+		(model "${KICAD9_3DMODEL_DIR}/Rotary_Encoder.3dshapes/RotaryEncoder_Alps_EC12E-Switch_Vertical_H20mm.step"
 			(offset
-				(xyz 7.5 -2.5 0)
+				(xyz 0 0 0)
 			)
 			(scale
@@
 			)
 			(rotate
-				(xyz -0 -0 90)
+				(xyz 0 0 0)
 			)
 		)
 	)
-	(footprint "Library:SW_Cherry_MX_1.00u_PCB_model"
+	(footprint "Button_Switch_Keyboard:SW_Cherry_MX_1.00u_PCB"
 		(layer "F.Cu")
 		(at 38.1 38.1)
@@
 			)
 		)
-		(property "Datasheet" ""
+		(property "Datasheet" "~"
 			(at 0 0 0)
 			(unlocked yes)
@@
 			)
 		)
-		(property "Description" ""
+		(property "Description" "Push button switch, normally open, two pins, 45° tilted"
 			(at 0 0 0)
 			(unlocked yes)
@@
 		)
 		(embedded_fonts no)
-		(model "${KICAD9_3DMODEL_DIR}/Button_Switch_THT.3dshapes/Cherry MX.STEP"
+		(model "${KICAD9_3DMODEL_DIR}/Button_Switch_Keyboard.3dshapes/SW_Cherry_MX_1.00u_PCB.step"
 			(offset
-				(xyz -2.5 -4 0)
+				(xyz 0 0 0)
 			)
 			(scale
@@
 			)
 			(rotate
-				(xyz -90 -0 -0)
+				(xyz 0 0 0)
 			)
 		)
 	)
-	(footprint "Library:SW_Cherry_MX_1.00u_PCB_model"
+	(footprint "Button_Switch_Keyboard:SW_Cherry_MX_1.00u_PCB"
 		(layer "F.Cu")
 		(at 76.2 57.15)
@@
 			)
 		)
-		(property "Datasheet" ""
+		(property "Datasheet" "~"
 			(at 0 0 0)
 			(unlocked yes)
@@
 			)
 		)
-		(property "Description" ""
+		(property "Description" "Push button switch, normally open, two pins, 45° tilted"
 			(at 0 0 0)
 			(unlocked yes)
@@
 		)
 		(embedded_fonts no)
-		(model "${KICAD9_3DMODEL_DIR}/Button_Switch_THT.3dshapes/Cherry MX.STEP"
+		(model "${KICAD9_3DMODEL_DIR}/Button_Switch_Keyboard.3dshapes/SW_Cherry_MX_1.00u_PCB.step"
 			(offset
-				(xyz -2.5 -4 0)
+				(xyz 0 0 0)
 			)
 			(scale
@@
 			)
 			(rotate
-				(xyz -90 -0 -0)
+				(xyz 0 0 0)
 			)
 		)
@@
 		)
 	)
-	(footprint "Library:SW_Cherry_MX_1.00u_PCB_model"
+	(footprint "Button_Switch_Keyboard:SW_Cherry_MX_1.00u_PCB"
 		(layer "F.Cu")
 		(at 76.2 38.1)
@@
 			)
 		)
-		(property "Datasheet" ""
+		(property "Datasheet" "~"
 			(at 0 0 0)
 			(unlocked yes)
@@
 			)
 		)
-		(property "Description" ""
+		(property "Description" "Push button switch, normally open, two pins, 45° tilted"
 			(at 0 0 0)
 			(unlocked yes)
@@
 		)
 		(embedded_fonts no)
-		(model "${KICAD9_3DMODEL_DIR}/Button_Switch_THT.3dshapes/Cherry MX.STEP"
+		(model "${KICAD9_3DMODEL_DIR}/Button_Switch_Keyboard.3dshapes/SW_Cherry_MX_1.00u_PCB.step"
 			(offset
-				(xyz -2.5 -4 0)
+				(xyz 0 0 0)
 			)
 			(scale
@@
 			)
 			(rotate
-				(xyz -90 -0 -0)
+				(xyz 0 0 0)
 			)
 		)
@@
 		)
 		(embedded_fonts no)
-		(model "C:/Kicad_Extra/OPL_Kicad_Library/Seeed Studio XIAO-ESP32-C3.step"
-			(offset
-				(xyz 6 -2 0)
-			)
-			(scale
-				(xyz 1 1 1)
-			)
-			(rotate
-				(xyz -90 -0 -90)
-			)
-		)
 	)
 	(footprint "Diode_THT:D_DO-27_P15.24mm_Horizontal"
@@
 		(embedded_fonts no)
 	)
-	(footprint "Library:SW_Cherry_MX_1.00u_PCB_model"
+	(footprint "Button_Switch_Keyboard:SW_Cherry_MX_1.00u_PCB"
 		(layer "F.Cu")
 		(at 38.1 57.15)
@@
 			)
 		)
-		(property "Datasheet" ""
+		(property "Datasheet" "~"
 			(at 0 0 0)
 			(unlocked yes)
@@
 			)
 		)
-		(property "Description" ""
+		(property "Description" "Push button switch, normally open, two pins, 45° tilted"
 			(at 0 0 0)
 			(unlocked yes)
@@
 		)
 		(embedded_fonts no)
-		(model "${KICAD9_3DMODEL_DIR}/Button_Switch_THT.3dshapes/Cherry MX.STEP"
+		(model "${KICAD9_3DMODEL_DIR}/Button_Switch_Keyboard.3dshapes/SW_Cherry_MX_1.00u_PCB.step"
 			(offset
-				(xyz -2.5 -4 0)
+				(xyz 0 0 0)
 			)
 			(scale
@@
 			)
 			(rotate
-				(xyz -90 -0 -0)
+				(xyz 0 0 0)
 			)
 		)
@@
 		(layer "Edge.Cuts")
 	)
+	(gr_rect
+		(start 195.5 52.25)
+		(end 209.5 66.25)
+		(stroke
+			(width 0.05)
+			(type default)
+		)
+		(fill no)
+		(layer "Edge.Cuts")
+	)
+	(gr_rect
+		(start 157.5 52.25)
+		(end 171.5 66.25)
+		(stroke
+			(width 0.05)
+			(type default)
+		)
+		(fill no)
+		(layer "Edge.Cuts")
+	)
+	(gr_rect
+		(start 176.5 52.25)
+		(end 190.5 66.25)
+		(stroke
+			(width 0.05)
+			(type default)
+		)
+		(fill no)
+		(layer "Edge.Cuts")
+	)
 	(gr_line
 		(start 24 31)
@@
 		(layer "Edge.Cuts")
 	)
+	(gr_rect
+		(start 195.5 33.25)
+		(end 209.5 47.25)
+		(stroke
+			(width 0.05)
+			(type default)
+		)
+		(fill no)
+		(layer "Edge.Cuts")
+	)
 	(gr_line
 		(start 25 74)
@@
 		(layer "Edge.Cuts")
 	)
+	(gr_rect
+		(start 176.5 33.25)
+		(end 190.5 47.25)
+		(stroke
+			(width 0.05)
+			(type default)
+		)
+		(fill no)
+		(layer "Edge.Cuts")
+	)
 	(gr_arc
 		(start 109 73)
@@
 		(layer "Edge.Cuts")
 	)
+	(gr_circle
+		(center 140.75 50.5)
+		(end 140.75 54.5)
+		(stroke
+			(width 0.05)
+			(type default)
+		)
+		(fill no)
+		(layer "Edge.Cuts")
+	)
 	(gr_line
 		(start 25 30)
@@
 		(layer "Edge.Cuts")
 	)
+	(gr_rect
+		(start 157.5 33.25)
+		(end 171.5 47.25)
+		(stroke
+			(width 0.05)
+			(type default)
+		)
+		(fill no)
+		(layer "Edge.Cuts")
+	)
