File: PCB/hackpad.kicad_sch (KiCad schematic)
At the start: 15 parts, among them SW1 SW_Push_45deg, SW2 SW_Push_45deg, SW3 SW_Push_45deg, SW4 SW_Push_45deg, SW5 SW_Push_45deg, SW6 SW_Push_45deg, SW7 RotaryEncoder_Switch, U1 MOUDLE-SEEEDUINO-XIAO

Commit message: code
Connections:
- net R0: now also D1.1 (K)
- net R1: now also D2.1 (K)
- net R2: now also D3.1 (K)
- net at D4.2 (A), SW4.2: no longer D1.1 (K)
- net at D6.2 (A), SW6.2: no longer D3.1 (K)
- net at D5.2 (A), SW5.2: no longer D2.1 (K)
Changed lines of the file:
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@@
-	)
-	(junction
-		(at 182.88 81.28)
-		(diameter 0)
-		(color 0 0 0 0)
-	)
-	(junction
-		(at 233.68 81.28)
-		(diameter 0)
-		(color 0 0 0 0)
 	)
 	(junction
@@
 		(color 0 0 0 0)
 	)
-	(junction
-		(at 208.28 81.28)
-		(diameter 0)
-		(color 0 0 0 0)
-	)
-	(wire
-		(pts
-			(xy 233.68 63.5) (xy 233.68 81.28)
+	(wire
+		(pts
+			(xy 208.28 63.5) (xy 210.82 63.5)
+		)
+		(stroke
+			(width 0)
+			(type default)
+		)
+	)
+	(wire
+		(pts
+			(xy 210.82 63.5) (xy 210.82 88.9)
+		)
+		(stroke
+			(width 0)
+			(type default)
+		)
+	)
+	(wire
+		(pts
+			(xy 184.15 63.5) (xy 184.15 88.9)
+		)
+		(stroke
+			(width 0)
+			(type default)
+		)
+	)
+	(wire
+		(pts
+			(xy 233.68 63.5) (xy 234.95 63.5)
 		)
 		(stroke
@@
 	(wire
 		(pts
+			(xy 210.82 88.9) (xy 208.28 88.9)
+		)
+		(stroke
+			(width 0)
+			(type default)
+		)
+	)
+	(wire
+		(pts
 			(xy 177.8 50.8) (xy 203.2 50.8)
 		)
@@
 	(wire
 		(pts
+			(xy 182.88 63.5) (xy 184.15 63.5)
+		)
+		(stroke
+			(width 0)
+			(type default)
+		)
+	)
+	(wire
+		(pts
+			(xy 234.95 63.5) (xy 234.95 88.9)
+		)
+		(stroke
+			(width 0)
+			(type default)
+		)
+	)
+	(wire
+		(pts
 			(xy 203.2 76.2) (xy 228.6 76.2)
 		)
@@
 	(wire
 		(pts
+			(xy 234.95 88.9) (xy 233.68 88.9)
+		)
+		(stroke
+			(width 0)
+			(type default)
+		)
+	)
+	(wire
+		(pts
 			(xy 138.43 111.76) (xy 138.43 110.49)
 		)
@@
 	(wire
 		(pts
-			(xy 182.88 63.5) (xy 182.88 81.28)
+			(xy 184.15 88.9) (xy 182.88 88.9)
 		)
 		(stroke
@@
 		)
 	)
-	(wire
-		(pts
-			(xy 208.28 63.5) (xy 208.28 81.28)
-		)
-		(stroke
-			(width 0)
-			(type default)
-		)
-	)
 	(global_label "C0"
 		(shape input)
@@
 		)
 	)
+	(global_label "R1"
+		(shape input)
+		(at 210.82 88.9 270)
+		(fields_autoplaced yes)
+		(effects
+			(font
+				(size 1.27 1.27)
+			)
+			(justify right)
+		)
+		(property "Intersheetrefs" "${INTERSHEET_REFS}"
+			(at 210.82 94.3647 90)
+			(effects
+				(font
+					(size 1.27 1.27)
+				)
+				(justify right)
+				(hide yes)
+			)
+		)
+	)
+	(global_label "R0"
+		(shape input)
+		(at 184.15 88.9 270)
+		(fields_autoplaced yes)
+		(effects
+			(font
+				(size 1.27 1.27)
+			)
+			(justify right)
+		)
+		(property "Intersheetrefs" "${INTERSHEET_REFS}"
+			(at 184.15 94.3647 90)
+			(effects
+				(font
+					(size 1.27 1.27)
+				)
+				(justify right)
+				(hide yes)
+			)
+		)
+	)
 	(global_label "R2"
 		(shape input)
-		(at 233.68 88.9 270)
-		(fields_autoplaced yes)
-		(effects
-			(font
-				(size 1.27 1.27)
-			)
-			(justify right)
-		)
-		(property "Intersheetrefs" "${INTERSHEET_REFS}"
-			(at 233.68 94.3647 90)
-			(effects
-				(font
-					(size 1.27 1.27)
-				)
-				(justify right)
-				(hide yes)
-			)
-		)
-	)
-	(global_label "R1"
-		(shape input)
-		(at 208.28 88.9 270)
-		(fields_autoplaced yes)
-		(effects
-			(font
-				(size 1.27 1.27)
-			)
-			(justify right)
-		)
-		(property "Intersheetrefs" "${INTERSHEET_REFS}"
-			(at 208.28 94.3647 90)
-			(effects
-				(font
-					(size 1.27 1.27)
-				)
-				(justify right)
-				(hide yes)
-			)
-		)
-	)
-	(global_label "R0"
-		(shape input)
-		(at 182.88 88.9 270)
-		(fields_autoplaced yes)
-		(effects
-			(font
-				(size 1.27 1.27)
-			)
-			(justify right)
-		)
-		(property "Intersheetrefs" "${INTERSHEET_REFS}"
-			(at 182.88 94.3647 90)
-			(effects
-				(font
+		(at 234.95 88.9 270)
+		(fields_autoplaced yes)
+		(effects
+			(font
+				(size 1.27 1.27)
+			)
+			(justify right)
+		)
+		(property "Intersheetrefs" "${INTERSHEET_REFS}"
+			(at 234.95 94.3647 90)
+			(effects
+				(font

Commit message: WORKING PIC
Parts:
- D1, D2, D3, D4, D5, D6: footprint Diode_THT:D_DO-27_P15.24mm_Horizontal -> Diode_THT:D_DO-35_SOD27_P7.62mm_Horizontal
Other:
- moved on the sheet: Brd1, SW7
Changed lines of the file:
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@@
 	(wire
 		(pts
-			(xy 138.43 111.76) (xy 138.43 110.49)
+			(xy 257.81 64.77) (xy 257.81 63.5)
 		)
 		(stroke
@@
 	(global_label "D8"
 		(shape input)
-		(at 143.51 95.25 0)
+		(at 262.89 48.26 0)
 		(fields_autoplaced yes)
 		(effects
@@
 		)
 		(property "Intersheetrefs" "${INTERSHEET_REFS}"
-			(at 148.9747 95.25 0)
+			(at 268.3547 48.26 0)
 			(effects
 				(font
@@
 	(global_label "SCL"
 		(shape input)
-		(at 99.06 96.52 90)
+		(at 91.44 64.77 90)
 		(fields_autoplaced yes)
 		(effects
@@
 		)
 		(property "Intersheetrefs" "${INTERSHEET_REFS}"
-			(at 99.06 90.0272 90)
+			(at 91.44 58.2772 90)
 			(effects
 				(font
@@
 	(global_label "SDA"
 		(shape input)
-		(at 101.6 96.52 90)
+		(at 93.98 64.77 90)
 		(fields_autoplaced yes)
 		(effects
@@
 		)
 		(property "Intersheetrefs" "${INTERSHEET_REFS}"
-			(at 101.6 89.9667 90)
+			(at 93.98 58.2167 90)
 			(effects
 				(font
@@
 	(global_label "D9"
 		(shape input)
-		(at 138.43 95.25 180)
+		(at 257.81 48.26 180)
 		(fields_autoplaced yes)
 		(effects
@@
 		)
 		(property "Intersheetrefs" "${INTERSHEET_REFS}"
-			(at 132.9653 95.25 0)
+			(at 252.3453 48.26 0)
 			(effects
 				(font
@@
 	(global_label "D10"
 		(shape input)
-		(at 138.43 111.76 180)
+		(at 257.81 64.77 180)
 		(fields_autoplaced yes)
 		(effects
@@
 		)
 		(property "Intersheetrefs" "${INTERSHEET_REFS}"
-			(at 131.7558 111.76 0)
+			(at 251.1358 64.77 0)
 			(effects
 				(font
@@
 	(symbol
 		(lib_id "SSD1306-128x64_OLED:SSD1306")
-		(at 97.79 105.41 0)
+		(at 90.17 73.66 0)
 		(unit 1)
 		(exclude_from_sim no)
@@
 		(fields_autoplaced yes)
 		(property "Reference" "Brd1"
-			(at 105.41 104.1399 0)
+			(at 97.79 72.3899 0)
 			(effects
 				(font
@@
 		)
 		(property "Value" "SSD1306"
-			(at 105.41 106.6799 0)
+			(at 97.79 74.9299 0)
 			(effects
 				(font
@@
 		)
 		(property "Footprint" "SSD1306:128x64OLED"
-			(at 97.79 99.06 0)
+			(at 90.17 67.31 0)
 			(effects
 				(font
@@
 		)
 		(property "Datasheet" ""
-			(at 97.79 99.06 0)
+			(at 90.17 67.31 0)
 			(effects
 				(font
@@
 		)
 		(property "Description" "SSD1306 OLED"
-			(at 97.79 105.41 0)
+			(at 90.17 73.66 0)
 			(effects
 				(font
@@
 	(symbol
 		(lib_id "power:GND")
-		(at 93.98 96.52 270)
+		(at 86.36 64.77 270)
 		(unit 1)
 		(exclude_from_sim no)
@@
 		(fields_autoplaced yes)
 		(property "Reference" "#PWR02"
-			(at 87.63 96.52 0)
+			(at 80.01 64.77 0)
 			(effects
 				(font
@@
 		)
 		(property "Value" "GND"
-			(at 90.17 96.5199 90)
+			(at 82.55 64.7699 90)
 			(effects
 				(font
@@
 		)
 		(property "Footprint" ""
-			(at 93.98 96.52 0)
+			(at 86.36 64.77 0)
 			(effects
 				(font
@@
 		)
 		(property "Datasheet" ""
-			(at 93.98 96.52 0)
+			(at 86.36 64.77 0)
 			(effects
 				(font
@@
 		)
 		(property "Description" "Power symbol creates a global label with name \"GND\" , ground"
-			(at 93.98 96.52 0)
+			(at 86.36 64.77 0)
 			(effects
 				(font
@@
 			)
 		)
-		(property "Footprint" "Diode_THT:D_DO-27_P15.24mm_Horizontal"
+		(property "Footprint" "Diode_THT:D_DO-35_SOD27_P7.62mm_Horizontal"
 			(at 233.68 59.69 0)
 			(effects
@@
 	(symbol
 		(lib_id "power:GND")
-		(at 143.51 110.49 0)
+		(at 262.89 63.5 0)
 		(unit 1)
 		(exclude_from_sim no)
@@
 		(fields_autoplaced yes)
 		(property "Reference" "#PWR05"
-			(at 143.51 116.84 0)
+			(at 262.89 69.85 0)
 			(effects
 				(font
@@
 		)
 		(property "Value" "GND"
-			(at 143.51 115.57 0)
+			(at 262.89 68.58 0)
 			(effects
 				(font
@@
 		)
 		(property "Footprint" ""
-			(at 143.51 110.49 0)
+			(at 262.89 63.5 0)
 			(effects
 				(font
@@
 		)
 		(property "Datasheet" ""
-			(at 143.51 110.49 0)
+			(at 262.89 63.5 0)
 			(effects
 				(font
@@
 		)
 		(property "Description" "Power symbol creates a global label with name \"GND\" , ground"
-			(at 143.51 110.49 0)
+			(at 262.89 63.5 0)
 			(effects
 				(font
@@
 	(symbol
 		(lib_id "Device:RotaryEncoder_Switch")
-		(at 140.97 102.87 270)
+		(at 260.35 55.88 270)
 		(unit 1)
 		(exclude_from_sim no)
@@
 		(fields_autoplaced yes)
 		(property "Reference" "SW7"
-			(at 147.32 101.5999 90)
+			(at 266.7 54.6099 90)
 			(effects
 				(font
@@
 		)
 		(property "Value" "RotaryEncoder_Switch"
-			(at 147.32 104.1399 90)
+			(at 266.7 57.1499 90)
 			(effects
 				(font
@@
 		)
 		(property "Footprint" "Rotary_Encoder:RotaryEncoder_Alps_EC12E-Switch_Vertical_H20mm"
-			(at 145.034 99.06 0)
+			(at 264.414 52.07 0)
 			(effects
 				(font
@@
 		)
 		(property "Datasheet" "~"
-			(at 147.574 102.87 0)
+			(at 266.954 55.88 0)
 			(effects
 				(font
@@
 		)
 		(property "Description" "Rotary encoder, dual channel, incremental quadrate outputs, with switch"
-			(at 140.97 102.87 0)
+			(at 260.35 55.88 0)
 			(effects
 				(font
@@
 	(symbol
 		(lib_id "power:GND")
-		(at 140.97 95.25 180)
+		(at 260.35 48.26 180)
 		(unit 1)
 		(exclude_from_sim no)
@@
 		(fields_autoplaced yes)
 		(property "Reference" "#PWR06"
-			(at 140.97 88.9 0)
+			(at 260.35 41.91 0)
 			(effects
 				(font
@@
 		)
 		(property "Value" "GND"
-			(at 140.97 90.17 0)
+			(at 260.35 43.18 0)
 			(effects
 				(font
@@
 		)
 		(property "Footprint" ""
-			(at 140.97 95.25 0)
+			(at 260.35 48.26 0)
 			(effects
 				(font
@@
 		)
 		(property "Datasheet" ""
-			(at 140.97 95.25 0)
+			(at 260.35 48.26 0)
 			(effects
 				(font
@@
 		)
 		(property "Description" "Power symbol creates a global label with name \"GND\" , ground"
-			(at 140.97 95.25 0)
+			(at 260.35 48.26 0)
 			(effects
 				(font
@@
 			)
 		)
-		(property "Footprint" "Diode_THT:D_DO-27_P15.24mm_Horizontal"
+		(property "Footprint" "Diode_THT:D_DO-35_SOD27_P7.62mm_Horizontal"
 			(at 182.88 85.09 0)
 			(effects
@@
 			)
 		)
-		(property "Footprint" "Diode_THT:D_DO-27_P15.24mm_Horizontal"
+		(property "Footprint" "Diode_THT:D_DO-35_SOD27_P7.62mm_Horizontal"
 			(at 208.28 59.69 0)
 			(effects
@@
 			)
 		)
-		(property "Footprint" "Diode_THT:D_DO-27_P15.24mm_Horizontal"
+		(property "Footprint" "Diode_THT:D_DO-35_SOD27_P7.62mm_Horizontal"
 			(at 182.88 59.69 0)
 			(effects
@@
 	(symbol
 		(lib_id "power:+5V")
-		(at 96.52 96.52 0)
+		(at 88.9 64.77 0)
 		(unit 1)
 		(exclude_from_sim no)
@@
 		(fields_autoplaced yes)
 		(property "Reference" "#PWR03"
-			(at 96.52 100.33 0)
+			(at 88.9 68.58 0)
 			(effects
 				(font
@@
 		)
 		(property "Value" "+5V"
-			(at 96.52 91.44 0)
+			(at 88.9 59.69 0)
 			(effects
 				(font
@@
 		)
 		(property "Footprint" ""
-			(at 96.52 96.52 0)
+			(at 88.9 64.77 0)
 			(effects
 				(font
@@
 		)
 		(property "Datasheet" ""
-			(at 96.52 96.52 0)
+			(at 88.9 64.77 0)
 			(effects
 				(font
@@
 		)
 		(property "Description" "Power symbol creates a global label with name \"+5V\""
-			(at 96.52 96.52 0)
+			(at 88.9 64.77 0)
 			(effects
 				(font
@@
 			)
 		)
-		(property "Footprint" "Diode_THT:D_DO-27_P15.24mm_Horizontal"
+		(property "Footprint" "Diode_THT:D_DO-35_SOD27_P7.62mm_Horizontal"
 			(at 208.28 85.09 0)
 			(effects
@@
 			)
 		)
-		(property "Footprint" "Diode_THT:D_DO-27_P15.24mm_Horizontal"
+		(property "Footprint" "Diode_THT:D_DO-35_SOD27_P7.62mm_Horizontal"
 			(at 233.68 85.09 0)
 			(effects
