File: PCB/hackpad.kicad_pcb (KiCad board)
At the start: 2 copper layers, 85 x 44 mm, 18 parts, among them SW1 SW_Push_45deg, SW2 SW_Push_45deg, SW3 SW_Push_45deg, SW4 SW_Push_45deg, SW5 SW_Push_45deg, SW6 SW_Push_45deg, SW7 RotaryEncoder_Switch, U1 MOUDLE-SEEEDUINO-XIAO

Commit message: code
Parts:
- removed REF** (x3): MountingHole_3.2mm_M3_ISO7380, MountingHole:MountingHole_3.2mm_M3_ISO7380
- SW1, SW2, SW3, SW4, SW5, SW6: footprint Library:SW_Cherry_MX_1.00u_PCB_model -> Button_Switch_Keyboard:SW_Cherry_MX_1.00u_PCB
Connections:
- D1 pad 1: Net-(D1-K) -> R0
- D2 pad 1: Net-(D2-K) -> R1
- D3 pad 1: Net-(D3-K) -> R2
- D4 pad 2: Net-(D1-K) -> Net-(D4-A)
- D5 pad 2: Net-(D2-K) -> Net-(D5-A)
- D6 pad 2: Net-(D3-K) -> Net-(D6-A)
- SW4 pad 2: Net-(D1-K) -> Net-(D4-A)
- SW5 pad 2: Net-(D2-K) -> Net-(D5-A)
- SW6 pad 2: Net-(D3-K) -> Net-(D6-A)
Routing:
- net Net-(D1-K): track 42.7 -> 0.00 mm
- net Net-(D3-K): track 42.7 -> 0.00 mm
- net Net-(D2-K): track 42.7 -> 0.00 mm
- net R2: track 30.1 -> 49.1 mm
- net R1: track 66.2 -> 85.3 mm
- net R0: track 78.7 -> 97.8 mm
- net Net-(D4-A): track 0.00 -> 16.3 mm
- net Net-(D5-A): track 0.00 -> 16.3 mm
- net Net-(D6-A): track 0.00 -> 16.3 mm

Commit message: WORKING PIC
Parts:
- added G***: LOGO, LOGO, F.Cu at (65.8, 51.5)
- added REF**: UKCA-Logo_6x6mm_SilkScreen, Symbol:UKCA-Logo_6x6mm_SilkScreen, B.Cu at (27.5, 53.0)
- added kibuzzard-69AC02E9: G***, kibuzzard-69AC02E9, F.Cu at (66.5, 32.0)
- added kibuzzard-69AC02E9: G***, kibuzzard-69AC02E9, B.Cu at (66.5, 32.0)
- added kibuzzard-69AC031A: G***, kibuzzard-69AC031A, F.Cu at (66.5, 32.0)
- added kibuzzard-69AC031A: G***, kibuzzard-69AC031A, B.Cu at (66.5, 32.0)
- added kibuzzard-69AC06C1: G***, kibuzzard-69AC06C1, B.Cu at (66.5, 53.5)
- moved U1 5.32 mm to (96.9, 40.4)
Routing:
- net R2: track 49.1 -> 53.8 mm, vias 1 -> 0
- net D9: track 16.2 -> 21.0 mm
- net D10: track 30.8 -> 35.5 mm
- net C1: track 64.8 -> 68.5 mm
- net D8: track 21.5 -> 25.2 mm
- net R0: track 97.8 -> 101.5 mm
- net SDA: track 24.1 -> 27.8 mm
- net SCL: track 21.5 -> 22.9 mm, vias 0 -> 1
- net R1: track 85.3 -> 86.4 mm
- net C0: track 52.3 -> 53.3 mm
Other:
- board text added: "${REFERENCE}"
- board text added: "K"

Commit message: Done
Parts:
- added REF**: MountingHole_2.5mm_Pad_TopBottom, MountingHole:MountingHole_2.5mm_Pad_TopBottom, F.Cu at (106.0, 71.0)
- added REF**: MountingHole_2.5mm_Pad_TopBottom, MountingHole:MountingHole_2.5mm_Pad_TopBottom, F.Cu at (96.9, 40.4)
- added REF**: MountingHole_2.5mm_Pad_TopBottom, MountingHole:MountingHole_2.5mm_Pad_TopBottom, F.Cu at (54.0, 51.5)
